File: hardware/kcan-rxonly-pcb/kicad/BMW-E9x-KCAN-RXOnly.kicad_pcb (KiCad board)
At the start: 2 copper layers, 120 x 80 mm, 50 parts, among them J1 J_BAT 10..18V BENCH, J2 J_KCAN H L GND, U1 TJA1055T/3/2Z, U2 CLVC1G125QDBVRQ1, U3 TLS715B0EJV50XUMA1

Commit message: hardware: optimize U3 thermal DFM
Parts:
- U3: footprint Infineon_PG-DSO-8-52_3.9x4.9mm_EP2.65x3mm_ThermalVias -> Infineon_PG-DSO-8-52_3.9x4.9mm_EP2.65x3mm_NoViaInPad
Routing:
- net GND: vias 3 -> 7
