File: hardware/kcan-rxonly-pcb/kicad/BMW-E9x-KCAN-RXOnly.kicad_sch (KiCad schematic)
At the start: 46 parts, among them J1 BENCH 10..18V / J_BAT, J2 LSFT BENCH BUS / J_KCAN, U1 TJA1055T/3/2Z, U2 CLVC1G125QDBVRQ1, U3 TLS715B0EJV50XUMA1

Commit message: hardware: optimize U3 thermal DFM
Parts:
- U3: footprint Phase3G:Infineon_PG-DSO-8-52_3.9x4.9mm_EP2.65x3mm_ThermalVias -> Phase3G:Infineon_PG-DSO-8-52_3.9x4.9mm_EP2.65x3mm_NoViaInPad
Changed lines of the file:
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@@
 			)
 		)
-		(property "Footprint" "Phase3G:Infineon_PG-DSO-8-52_3.9x4.9mm_EP2.65x3mm_ThermalVias"
+		(property "Footprint" "Phase3G:Infineon_PG-DSO-8-52_3.9x4.9mm_EP2.65x3mm_NoViaInPad"
 			(at 44.45 85.09 0.0000)
 			(effects
